File: schem/schem.kicad_sch (KiCad schematic)
At the start: 11 parts

Commit message: schem updated
Parts:
- removed D1: IR204A, LED_THT:LED_D3.0mm_IRBlack, symbol LED:IR204A
- removed D2: LED_BRGK, symbol Device:LED_BRGK
- removed D3: D_Photo, symbol Device:D_Photo
- removed R1: 10kohm, symbol Device:R
- removed R2: R_Photo, symbol Device:R_Photo
- removed R3, R4, R5, R6: 100ohm, symbol Device:R
- removed R7: 500kohm, symbol Device:R
- added C1: 10uF, symbol Device:C
- added D1: LED_RGBA, symbol Device:LED_RGBA
- added R1: R_Photo, symbol Device:R_Photo
- added RV1, RV2: R_Potentiometer, symbol Device:R_Potentiometer
- added SW1, SW2, SW3: SW_SPST, symbol Switch:SW_SPST
Connections:
- net +3V3: now also RV1.1
- net GND: now also C1.2, R1.2, SW1.1 (A), SW2.1 (A), SW3.1 (A)
- net at A1.6 (D3): now also RV2.3
- net at A1.19 (A0): now also C1.1, R1.1, RV1.3
- new net: D1.1 (RK), SW1.2 (B)
- new net: D1.4 (A), RV2.1
- new net: D1.2 (GK), SW2.2 (B)
- new net: D1.3 (BK), SW3.2 (B)
